Commit message: Update Simulation

File: val2sim_model/sensors/ydlidar/ydlidar_g4.xacro (robot description, xacro)
@@ -13,5 +13,5 @@
                 <origin xyz="0 0 0" rpy="0 0 0"/>
                 <geometry>
-                    <mesh filename="package://val2_model/sensors/ydlidar/meshes/ydlidar_g4.dae" />
+                    <mesh filename="package://val2sim_model/sensors/ydlidar/meshes/ydlidar_g4.dae" />
                 </geometry>
                 <material name="light_black"/>
@@ -21,5 +21,5 @@
                 <geometry>
                     <cylinder length="0.05" radius="0.040"/>
-                    <!-- <mesh filename="package://val2_model/sensors/ydlidar/meshes/ydlidar_g4.dae" /> -->
+                    <!-- <mesh filename="package://val2sim_model/sensors/ydlidar/meshes/ydlidar_g4.dae" /> -->
                 </geometry>
             </collision>
