Commit message: Update Description

File: val2sim_description/urdf/val2sim.urdf (robot description, URDF)
Before this commit: robot val2sim, 6 links, 5 joints
Links:
- link base_link: geometry collision box size=0.46 0.6 0.14; collision sphere radius=0.0635
- link laser_base_link: geometry collision cylinder length=0.05 radius=0.040; visual mesh filename=package://val2_model/sensors/ydlidar/meshes/ydlidar_g4.dae
Joints:
- joint left_wheel_joint: origin xyz=-0.125 0.202 -0.005 rpy=0 0 0 -> xyz=0.0 0.307 -0.005 rpy=0 0 0
- joint right_wheel_joint: origin xyz=-0.125 -0.202 -0.005 rpy=0 0 0 -> xyz=0.0 -0.307 -0.005 rpy=0 0 0

File: val2sim_description/urdf/val2sim.xacro (robot description, xacro)
@@ -5,12 +5,12 @@
   <xacro:include filename="$(find val2sim_model)/sensors/ydlidar/ydlidar_g4.xacro"/>
   <xacro:include filename="$(find val2sim_gazebo)/plugins/val2_diffdrive_plugins.xacro"/>
-  <xacro:property name="base_width" value="0.39"/>
-  <xacro:property name="base_len" value="0.43"/>
+  <xacro:property name="base_width" value="0.60"/>
+  <xacro:property name="base_len" value="0.46"/>
   <xacro:property name="wheel_radius" value="0.075"/>
   <xacro:property name="base_wheel_gap" value="0.007"/>
   <xacro:property name="wheel_separation" value="0.355"/>
-  <xacro:property name="wheel_joint_offset" value="-0.125"/>
-  <xacro:property name="caster_wheel_radius" value="0.0225"/>
-  <xacro:property name="caster_z_offset" value="-0.06"/>
+  <xacro:property name="wheel_joint_offset" value="0.0"/>
+  <xacro:property name="caster_wheel_radius" value="0.0635"/>
+  <xacro:property name="caster_z_offset" value="-0.01640"/>
   <xacro:property name="caster_wheel_joint_offset" value="0.00"/>
   <xacro:macro name="box_inertia" params="m w h d">
@@ -50,6 +50,6 @@
       </geometry>
     </collision>
-    <collision name="caster_front1_collision">
-        <origin rpy="0 0 0" xyz="0.175 -0.085 ${caster_z_offset}"/>
+    <collision name="caster_front_collision">
+        <origin rpy="0 0 0" xyz="0.150 0.0 ${caster_z_offset}"/>
         <geometry>
           <sphere radius="${caster_wheel_radius}"/>
@@ -66,6 +66,6 @@
         </surface>
     </collision>
-    <visual name="caster_front1_visual">
-        <origin rpy=" 0 0 0" xyz="0.175 -0.085 ${caster_z_offset}"/>
+    <visual name="caster_front_visual">
+        <origin rpy=" 0 0 0" xyz="0.150 0.0 ${caster_z_offset}"/>
         <geometry>
           <sphere radius="${caster_wheel_radius}"/>
@@ -73,6 +73,6 @@
         <material name="black"/>
     </visual>
-    <collision name="caster_front2_collision">
-      <origin rpy="0 0 0" xyz="0.175 0.085 ${caster_z_offset}"/>
+    <collision name="caster_back_collision">
+      <origin rpy="0 0 0" xyz="-0.150 0.0 ${caster_z_offset}"/>
       <geometry>
         <sphere radius="${caster_wheel_radius}"/>
@@ -89,6 +89,6 @@
       </surface>
     </collision>
-    <visual name="caster_front2_visual">
-      <origin rpy="0 0 0" xyz="0.175 0.085 ${caster_z_offset}"/>
+    <visual name="caster_back_visual">
+      <origin rpy="0 0 0" xyz="-0.150 0.0 ${caster_z_offset}"/>
       <geometry>
         <sphere radius="${caster_wheel_radius}"/>

Commit message: Update Simulation

File: val2sim_description/urdf/val2sim.urdf (robot description, URDF)
Before this commit: robot val2sim, 6 links, 5 joints
Joints:
- joint base_link_joint: origin xyz=0.125 0 0.075 rpy=0 0 0 -> xyz=0.0 0 0.075 rpy=0 0 0
- joint laser_base_fixed: origin xyz=-0.05 0 0.14 rpy=0 0 0 -> xyz=0.15 0 0.10 rpy=0 0 0

File: val2sim_description/urdf/val2sim.xacro (robot description, xacro)
@@ -21,5 +21,4 @@
   </xacro:macro>
   <link name="base_footprint">
-    <!-- <xacro:box_inertia m="20" w="0.001" h="0.001" d="0.001"/> -->
     <visual>
         <origin xyz="0 0 0" rpy="0 0 0" />
@@ -96,30 +95,7 @@
       <material name="black"/>
     </visual>
-    <!-- <collision name="caster_back_collision">
-      <origin rpy="0 0 0" xyz="-0.04 0.0 ${caster_z_offset}"/>
-      <geometry>
-        <sphere radius="${caster_wheel_radius}"/>
-      </geometry>
-      <surface>
-        <friction>
-          <ode>
-            <mu>0</mu>
-            <mu2>0</mu2>
-            <slip1>1.0</slip1>
-            <slip2>1.0</slip2>
-          </ode>
-        </friction>
-      </surface>
-    </collision>
-    <visual name="caster_back_visual">
-      <origin rpy="0 0 0" xyz="-0.04 0.0 ${caster_z_offset}"/>
-      <geometry>
-        <sphere radius="${caster_wheel_radius}"/>
-      </geometry>
-      <material name="black"/>
-    </visual> -->
   </link>
   <joint name="base_link_joint" type="fixed">
-    <origin xyz="0.125 0 ${wheel_radius}" rpy="0 0 0" />
+    <origin xyz="0.0 0 ${wheel_radius}" rpy="0 0 0" />
     <parent link="base_footprint"/>
     <child link="base_link" />
@@ -163,28 +139,6 @@
     </inertial>
   </xacro:macro>
-  <!-- <link name="caster_wheel">
-    <visual>
-      <origin xyz="-0.070 0 0" rpy="0 0 0"/>
-      <geometry>
-        <sphere radius="${caster_wheel_radius}"/>
-      </geometry>
-      <material name="red"/>
-    </visual>
-    <collision>
-      <origin xyz="-0.070 0 0" rpy="0 0 0"/>
-      <geometry>
-        <sphere radius="${caster_wheel_radius}"/>
-      </geometry>
-    </collision>
-    <xacro:sphere_inertia m="5" r="${caster_wheel_radius}"/>
-  </link> -->
-  <!-- <joint name="caster_wheel_joint" type="continuous">
-    <axis xyz="0 1 0" rpy="0 0 0" />
-    <parent link="base_link"/>
-    <child link="caster_wheel"/>
-    <origin xyz="${caster_wheel_joint_offset} 0 -${caster_wheel_radius+0.005}" rpy="0 0 0"/>
-  </joint> -->
   <xacro:ydlidar_g4 prefix="laser" parent="base_link" prefix_topic='' visual='true' min_angle="-${PI}" max_angle="${PI}" min_range="0.26" max_range="12.0">
-    <origin xyz="-0.05 0 0.14" rpy="0 0 0"/>
+    <origin xyz="0.15 0 0.10" rpy="0 0 0"/>
   </xacro:ydlidar_g4>
 </robot>

File: val2sim_gazebo/plugins/val2_diffdrive_plugins.xacro (robot description, xacro)
@@ -2,6 +2,6 @@
 <robot
   xmlns:xacro="http://ros.org/wiki/xacro">
-  <xacro:property name="wheel_radius" value="0.035"/>
-  <xacro:property name="wheel_separation" value="0.15"/>
+  <xacro:property name="wheel_radius" value="0.075"/>
+  <xacro:property name="wheel_separation" value="0.355"/>
   <gazebo>
     <plugin name="differential_drive_controller" filename="libgazebo_ros_diff_drive.so">

Commit message: Update Simulation

File: val2sim_description/urdf/val2sim.urdf (robot description, URDF)
Before this commit: robot val2sim, 6 links, 5 joints
Links:
- link laser_base_link: geometry collision cylinder length=0.05 radius=0.040; visual mesh filename=package://val2sim_model/sensors/ydlidar/meshes/ydlidar_g4.d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

Commit message: Update Simulation

File: val2sim_description/urdf/val2sim.urdf (robot description, URDF)
Before this commit: robot val2sim, 6 links, 5 joints
Joints:
- joint left_wheel_joint: origin xyz=0.0 0.307 -0.005 rpy=0 0 0 -> xyz=0.0 0.2695 -0.005 rpy=0 0 0
- joint right_wheel_joint: origin xyz=0.0 -0.307 -0.005 rpy=0 0 0 -> xyz=0.0 -0.2695 -0.005 rpy=0 0 0

File: val2sim_description/urdf/val2sim.xacro (robot description, xacro)
@@ -9,5 +9,5 @@
   <xacro:property name="wheel_radius" value="0.075"/>
   <xacro:property name="base_wheel_gap" value="0.007"/>
-  <xacro:property name="wheel_separation" value="0.355"/>
+  <xacro:property name="wheel_separation" value="0.525"/>
   <xacro:property name="wheel_joint_offset" value="0.0"/>
   <xacro:property name="caster_wheel_radius" value="0.0635"/>
@@ -128,5 +128,6 @@
       <parent link="base_link"/>
       <child link="${prefix}_wheel"/>
-      <origin xyz="${wheel_joint_offset} ${((base_width/2)+base_wheel_gap)*reflect} -0.005" rpy="0 0 0"/>
+      <!-- <origin xyz="${wheel_joint_offset} ${((base_width/2)+base_wheel_gap)*reflect} -0.005" rpy="0 0 0"/> -->
+      <origin xyz="${wheel_joint_offset} ${((wheel_separation/2)+base_wheel_gap)*reflect} -0.005" rpy="0 0 0"/>
     </joint>
   </xacro:macro>

File: val2sim_gazebo/plugins/val2_diffdrive_plugins.xacro (robot description, xacro)
@@ -3,5 +3,5 @@
   xmlns:xacro="http://ros.org/wiki/xacro">
   <xacro:property name="wheel_radius" value="0.075"/>
-  <xacro:property name="wheel_separation" value="0.355"/>
+  <xacro:property name="wheel_separation" value="0.525"/>
   <gazebo>
     <plugin name="differential_drive_controller" filename="libgazebo_ros_diff_drive.so">

Commit message: Add comment

File: val2sim_description/urdf/val2sim.urdf (robot description, URDF)
Before this commit: robot val2sim, 6 links, 5 joints
Links:
- link left_wheel: geometry collision cylinder length=0.035 radius=0.090; visual cylinder length=0.035 radius=0.090
- link right_wheel: geometry collision cylinder length=0.035 radius=0.090; visual cylinder length=0.035 radius=0.090
Joints:
- joint base_link_joint: origin xyz=0.0 0 0.075 rpy=0 0 0 -> xyz=0.0 0 0.090 rpy=0 0 0
- joint left_wheel_joint: origin xyz=0.0 0.2695 -0.005 rpy=0 0 0 -> xyz=0.0 0.267 -0.005 rpy=0 0 0
- joint right_wheel_joint: origin xyz=0.0 -0.2695 -0.005 rpy=0 0 0 -> xyz=0.0 -0.267 -0.005 rpy=0 0 0

File: val2sim_description/urdf/val2sim.xacro (robot description, xacro)
@@ -7,7 +7,7 @@
   <xacro:property name="base_width" value="0.60"/>
   <xacro:property name="base_len" value="0.46"/>
-  <xacro:property name="wheel_radius" value="0.075"/>
+  <xacro:property name="wheel_radius" value="0.090"/>
   <xacro:property name="base_wheel_gap" value="0.007"/>
-  <xacro:property name="wheel_separation" value="0.525"/>
+  <xacro:property name="wheel_separation" value="0.534"/>
   <xacro:property name="wheel_joint_offset" value="0.0"/>
   <xacro:property name="caster_wheel_radius" value="0.0635"/>

Commit message: Update

File: val2sim_description/urdf/val2sim.urdf (robot description, URDF)
Before this commit: robot val2sim, 6 links, 5 joints
Links:
- link base_link: geometry collision box size=0.46 0.6 0.14; collision sphere radius=0.0785
- link left_wheel: geometry collision cylinder length=0.035 radius=0.09; visual cylinder length=0.035 radius=0.09
- link right_wheel: geometry collision cylinder length=0.035 radius=0.09; visual cylinder length=0.035 radius=0.09
Joints:
- joint base_link_joint: origin xyz=0.0 0 0.090 rpy=0 0 0 -> xyz=0.0 0 0.09 rpy=0 0 0
- joint left_wheel_joint: origin xyz=0.0 0.267 -0.005 rpy=0 0 0 -> xyz=0.0 0.274 -0.005 rpy=0 0 0
- joint right_wheel_joint: origin xyz=0.0 -0.267 -0.005 rpy=0 0 0 -> xyz=0.0 -0.274 -0.005 rpy=0 0 0

File: val2sim_description/urdf/val2sim.xacro (robot description, xacro)
@@ -11,5 +11,5 @@
   <xacro:property name="wheel_separation" value="0.534"/>
   <xacro:property name="wheel_joint_offset" value="0.0"/>
-  <xacro:property name="caster_wheel_radius" value="0.0635"/>
+  <xacro:property name="caster_wheel_radius" value="0.0785"/>
   <xacro:property name="caster_z_offset" value="-0.01640"/>
   <xacro:property name="caster_wheel_joint_offset" value="0.00"/>

Commit message: Update

File: val2sim_description/urdf/val2sim.urdf (robot description, URDF)
Before this commit: robot val2sim, 6 links, 5 joints
Links:
- link base_link: geometry collision box size=0.46 0.6 0.14; collision sphere radius=0.0635
- link left_wheel: geometry collision cylinder length=0.035 radius=0.075; visual cylinder length=0.035 radius=0.075
- link right_wheel: geometry collision cylinder length=0.035 radius=0.075; visual cylinder length=0.035 radius=0.075
Joints:
- joint base_link_joint: origin xyz=0.0 0 0.09 rpy=0 0 0 -> xyz=0.0 0 0.075 rpy=0 0 0
- joint left_wheel_joint: origin xyz=0.0 0.274 -0.005 rpy=0 0 0 -> xyz=0.0 0.2695 -0.005 rpy=0 0 0
- joint right_wheel_joint: origin xyz=0.0 -0.274 -0.005 rpy=0 0 0 -> xyz=0.0 -0.2695 -0.005 rpy=0 0 0

File: val2sim_description/urdf/val2sim.xacro (robot description, xacro)
@@ -7,9 +7,9 @@
   <xacro:property name="base_width" value="0.60"/>
   <xacro:property name="base_len" value="0.46"/>
-  <xacro:property name="wheel_radius" value="0.090"/>
+  <xacro:property name="wheel_radius" value="0.075"/>
   <xacro:property name="base_wheel_gap" value="0.007"/>
-  <xacro:property name="wheel_separation" value="0.534"/>
+  <xacro:property name="wheel_separation" value="0.525"/>
   <xacro:property name="wheel_joint_offset" value="0.0"/>
-  <xacro:property name="caster_wheel_radius" value="0.0785"/>
+  <xacro:property name="caster_wheel_radius" value="0.0635"/>
   <xacro:property name="caster_z_offset" value="-0.01640"/>
   <xacro:property name="caster_wheel_joint_offset" value="0.00"/>
